Commit message: Fixed tf_remove_child_frames node to latch on static topic, changed mir100 urdf to work with gazebo

File: mir_description/urdf/include/mir_100_v1.urdf.xacro (robot description, xacro)
@@ -1,137 +1,9 @@
-<?xml version="1.0"?>
-<robot xmlns:xacro="http://ros.org/wiki/xacro">
-  <xacro:include filename="$(find mir_description)/urdf/include/common_properties.urdf.xacro" />
-  <xacro:include filename="$(find mir_description)/urdf/include/imu.gazebo.urdf.xacro" />
-  <xacro:include filename="$(find mir_description)/urdf/include/mir_100.gazebo.xacro" />
-  <xacro:include filename="$(find mir_description)/urdf/include/mir_100.transmission.xacro" />
-  <xacro:include filename="$(find mir_description)/urdf/include/sick_s300.urdf.xacro" />
-  <xacro:include filename="$(find mir_description)/urdf/include/wheel.urdf.xacro" />
-  <xacro:include filename="$(find mir_description)/urdf/include/caster.urdf.xacro" />
-  <xacro:property name="deg_to_rad" value="0.017453293" />
-  <!-- The inertia for the MiR platform is intentionally chosen to be smaller than
-       the bounding box and also shifted a bit to the back, because most of the mass
-       is in the lower center back (because of the batteries). -->
-  <xacro:property name="mir_base_inertial_x" value="-0.05" />
-  <xacro:property name="mir_base_inertial_y" value="0.0" />
-  <xacro:property name="mir_base_inertial_z" value="0.15" />
-  <xacro:property name="mir_base_inertial_x_length" value="0.50" />
-  <xacro:property name="mir_base_inertial_y_length" value="0.30" />
-  <xacro:property name="mir_base_inertial_z_length" value="0.20" />
-  <xacro:property name="mir_100_act_wheel_radius" value="0.0625" />
-  <xacro:property name="mir_100_act_wheel_width" value="0.032" />
-  <xacro:property name="mir_100_act_wheel_mass" value="1.0" />
-  <xacro:property name="mir_100_act_wheel_dx" value="0.037646" />
-  <xacro:property name="mir_100_act_wheel_dy" value="0.222604" />
-  <xacro:property name="mir_100_caster_wheel_radius" value="${mir_100_act_wheel_radius}" />
-  <xacro:property name="mir_100_caster_wheel_width" value="${mir_100_act_wheel_width}" />
-  <xacro:property name="mir_100_caster_wheel_mass" value="${mir_100_act_wheel_mass}" />
-  <xacro:property name="mir_100_caster_wheel_dx" value="-0.0382" />
-  <xacro:property name="mir_100_caster_wheel_dy" value="0" />
-  <xacro:property name="mir_100_caster_wheel_dz" value="-0.094" />
-  <xacro:property name="mir_100_front_caster_wheel_base_dx" value="0.341346" />
-  <xacro:property name="mir_100_back_caster_wheel_base_dx" value="-0.270154" />
-  <xacro:property name="mir_100_caster_wheel_base_dy" value="0.203" />
-  <xacro:property name="mir_100_caster_wheel_base_dz" value="${mir_100_caster_wheel_radius-mir_100_caster_wheel_dz}" />
-  <!-- MiR 100 complete mass 78.2kg (8.2kg battery) -->
-  <!-- - 2x2kg sick laser = 4kg-->
-  <!-- - 4x caster wheels + rotation link: 4x 1.31 kg -->
-  <!-- - 2x act wheels: 2kg -->
-  <xacro:property name="mir_100_base_mass" value="66.96" />
-  <xacro:property name="imu_stdev" value="0.00017" />
-  <xacro:macro name="mir_100" params="prefix ns">
-    <link name="${prefix}base_footprint" />
-    <joint name="${prefix}base_joint" type="fixed">
-      <parent link="${prefix}base_footprint" />
-      <child link="${prefix}base_link" />
-      <origin xyz="0 0 0" rpy="0 0 0" />
-    </joint>
-    <link name="${prefix}base_link">
-      <xacro:box_inertial mass="${mir_100_base_mass}" x="${mir_base_inertial_x_length}" y="${mir_base_inertial_y_length}" z="${mir_base_inertial_z_length}">
-        <origin xyz="${mir_base_inertial_x + mir_100_act_wheel_dx} ${mir_base_inertial_y} ${mir_base_inertial_z}" rpy="0 0 0" />
-      </xacro:box_inertial>
-      <visual>
-        <origin xyz="${mir_100_act_wheel_dx} 0 0" rpy="0 0 0" />
-        <geometry>
-          <mesh filename="package://mir_description/meshes/visual/mir_100_base.stl" />
-        </geometry>
-        <xacro:insert_block name="material_white" />
-      </visual>
-      <collision>
-        <origin xyz="${mir_100_act_wheel_dx} 0 0" rpy="0 0 0" />
-        <geometry>
-          <mesh filename="package://mir_description/meshes/collision/mir_100_base.stl" />
-        </geometry>
-      </collision>
-    </link>
-    <gazebo reference="${prefix}base_link">
-      <material>Gazebo/White</material>
-    </gazebo>
-    <!-- IMU -->
-    <joint name="${prefix}base_link_to_imu_joint" type="fixed">
-      <parent link="${prefix}base_link" />
-      <child link="${prefix}imu_link" />
-      <origin xyz="0.0 0.0 0.25" rpy="0 0 0" />  <!-- same as real MiR -->
-    </joint>
-    <link name="${prefix}imu_link" />
-    <xacro:imu_gazebo link="${prefix}imu_link" imu_topic="${prefix}imu_data" update_rate="50.0" stdev="${imu_stdev}" />
-    <!-- Create an alias for imu_link. This is necessary because the real MiR's
-         TF has imu_link, but the imu_data topic is published in the imu_frame
-         frame. -->
-    <joint name="${prefix}imu_link_to_imu_frame_joint" type="fixed">
-      <parent link="${prefix}imu_link" />
-      <child link="${prefix}imu_frame" />
-      <origin xyz="0 0 0" rpy="0 0 0" />
-    </joint>
-    <link name="${prefix}imu_frame" />
-    <!-- Laser scanners -->
-    <!-- virtual link for merged laserscan-->
-    <joint name="${prefix}base_link_to_virtual_laser_joint" type="fixed">
-      <parent link="${prefix}base_link" />
-      <child link="${prefix}virtual_laser_link" />
-      <origin xyz="0.0 0.0 0.25" rpy="0.0 0.0 0" />
-    </joint>
-    <link name="${prefix}virtual_laser_link">
-    </link>
-    <joint name="${prefix}base_link_to_front_laser_joint" type="fixed">
-      <parent link="${prefix}base_link" />
-      <child link="${prefix}front_laser_link" />
-      <origin xyz="0.4288 0.2358 0.1914" rpy="0.0 0.0 ${0.25 * pi}" />  <!-- from visually matching up the meshes of the MiR and the laser scanner -->
-    </joint>
-    <xacro:sick_s300 prefix="${prefix}" link="front_laser_link" topic="f_scan" />
-    <joint name="${prefix}base_link_to_back_laser_joint" type="fixed">
-      <parent link="${prefix}base_link" />
-      <child link="${prefix}back_laser_link" />
-      <origin xyz="-0.3548 -0.2352 0.1914" rpy="0.0 0.0 ${-0.75 * pi}" />  <!-- from visually matching up the meshes of the MiR and the laser scanner -->
-    </joint>
-    <xacro:sick_s300 prefix="${prefix}" link="back_laser_link" topic="b_scan" />
-    <!-- Ultrasound sensors -->
-    <joint name="${prefix}us_1_joint" type="fixed">   <!-- right ultrasound -->
-      <parent link="${prefix}base_link" />
-      <child link="${prefix}us_1_frame" />
-      <origin xyz="0.45 -0.12 0.16 " rpy="0 0 0" />  <!-- from visually matching to the mesh of the MiR -->
-    </joint>
-    <link name="${prefix}us_1_frame" />
-    <joint name="${prefix}us_2_joint" type="fixed">   <!-- left ultrasound -->
-      <parent link="${prefix}base_link" />
-      <child link="${prefix}us_2_frame" />
-      <origin xyz="0.45 0.12 0.16 " rpy="0 0 0" />  <!-- from visually matching to the mesh of the MiR -->
-    </joint>
-    <link name="${prefix}us_2_frame" />
-    <!-- wheels -->
-    <xacro:actuated_wheel prefix="${prefix}" locationprefix="left" locationright="-1"/>
-    <xacro:actuated_wheel prefix="${prefix}" locationprefix="right" locationright="1"/>
-    <xacro:caster_wheel prefix="${prefix}" ns="${ns}" locationprefix="fl" locationright="-1" wheel_base_dx="${mir_100_front_caster_wheel_base_dx}"/>
-    <xacro:caster_wheel prefix="${prefix}" ns="${ns}" locationprefix="fr" locationright="1" wheel_base_dx="${mir_100_front_caster_wheel_base_dx}"/>
-    <xacro:caster_wheel prefix="${prefix}" ns="${ns}" locationprefix="bl" locationright="-1" wheel_base_dx="${mir_100_back_caster_wheel_base_dx}"/>
-    <xacro:caster_wheel prefix="${prefix}" ns="${ns}" locationprefix="br" locationright="1" wheel_base_dx="${mir_100_back_caster_wheel_base_dx}"/>
-    <joint name="${prefix}base_link_surface_joint" type="fixed">
-      <origin xyz="${mir_100_act_wheel_dx} 0 0.352" rpy="0 0 0" />
-      <parent link="${prefix}base_link" />
-      <child link="${prefix}surface" />
-      <axis xyz="0 0 1" />
-    </joint>
-    <link name="${prefix}surface"/>
-    <xacro:mir_100_wheel_transmissions prefix="${prefix}"/>
-    <xacro:p3d_base_controller prefix="${prefix}"/>
+<?xml version="1.0" ?>
+<robot xmlns:xacro="http://www.ros.org/wiki/xacro"
+       name="mir_100" >
+<!-- This file is only for backward compatibility before the "mir_100" to "mir" rename. -->
+  <xacro:include filename="$(find mir_description)/urdf/include/mir_v1.urdf.xacro" />
+  <xacro:macro name="mir_100" params="prefix">
+    <xacro:mir prefix="${prefix}" />
   </xacro:macro>
 </robot>
